File: matrix_low_side_drive.kicad_sch (KiCad schematic)
At the start: 20 parts, among them U17 BCR421_SOT26, U18 BCR421_SOT26, U19 BCR421_SOT26, U20 BCR421_SOT26, U21 BCR421_SOT26, U22 BCR421_SOT26, U23 BCR421_SOT26, U24 BCR421_SOT26, U25 BCR421_SOT26, U26 BCR421_SOT26

Commit message: [#72447] SCH: Update matrix drive resistors
Signed-off-by: Dawid Lentka <dlentka@antmicro.com>
Parts:
- R49, R50, R51, R52, R53, R54, R55, R56, R57, R58: value R_120R_0402 -> R_120R_0603; footprint antmicro-footprints:R_0402_1005Metric -> antmicro-footprints:R_0603_1608Metric; symbol antmicroResistors0402:R_120R_0402 -> antmicroResistors0603:R_120R_0603; MPN CR0402-FX-1200GLF -> CR0603-FX-1200ELF
Changed lines of the file:
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@@
 	(title_block
 		(title "LED Panel Board")
-		(date "2025-01-31")
+		(date "2025-02-04")
 		(rev "1.0.0")
 	)
@@
 	)
 	(symbol
-		(lib_id "antmicroResistors0402:R_120R_0402")
+		(lib_id "antmicroResistors0603:R_120R_0603")
 		(at 218.44 111.76 270)
 		(mirror x)
@@
 			)
 		)
-		(property "Value" "R_120R_0402"
+		(property "Value" "R_120R_0603"
 			(at 205.74 91.44 0)
 			(effects
@@
 			)
 		)
-		(property "Footprint" "antmicro-footprints:R_0402_1005Metric"
+		(property "Footprint" "antmicro-footprints:R_0603_1608Metric"
 			(at 203.2 91.44 0)
 			(effects
@@
 			)
 		)
-		(property "Description" "SMD Chip Resistor, 120 ohm, ± 1%, 63 mW, 0402 [1005 Metric], Thick Film, General Purpose"
+		(property "Description" "SMD Chip Resistor, 120 ohm, ± 1%, 100 mW, 0603 [1608 Metric], Thick Film, General Purpose"
 			(at 218.44 111.76 0)
 			(effects
@@
 			)
 		)
-		(property "MPN" "CR0402-FX-1200GLF"
+		(property "MPN" "CR0603-FX-1200ELF"
 			(at 198.12 91.44 0)
 			(effects
@@
 	)
 	(symbol
-		(lib_id "antmicroResistors0402:R_120R_0402")
+		(lib_id "antmicroResistors0603:R_120R_0603")
 		(at 104.14 66.04 270)
 		(mirror x)
@@
 			)
 		)
-		(property "Value" "R_120R_0402"
+		(property "Value" "R_120R_0603"
 			(at 91.44 45.72 0)
 			(effects
@@
 			)
 		)
-		(property "Footprint" "antmicro-footprints:R_0402_1005Metric"
+		(property "Footprint" "antmicro-footprints:R_0603_1608Metric"
 			(at 88.9 45.72 0)
 			(effects
@@
 			)
 		)
-		(property "Description" "SMD Chip Resistor, 120 ohm, ± 1%, 63 mW, 0402 [1005 Metric], Thick Film, General Purpose"
+		(property "Description" "SMD Chip Resistor, 120 ohm, ± 1%, 100 mW, 0603 [1608 Metric], Thick Film, General Purpose"
 			(at 104.14 66.04 0)
 			(effects
@@
 			)
 		)
-		(property "MPN" "CR0402-FX-1200GLF"
+		(property "MPN" "CR0603-FX-1200ELF"
 			(at 83.82 45.72 0)
 			(effects
@@
 	)
 	(symbol
-		(lib_id "antmicroResistors0402:R_120R_0402")
+		(lib_id "antmicroResistors0603:R_120R_0603")
 		(at 218.44 66.04 270)
 		(mirror x)
@@
 			)
 		)
-		(property "Value" "R_120R_0402"
+		(property "Value" "R_120R_0603"
 			(at 205.74 45.72 0)
 			(effects
@@
 			)
 		)
-		(property "Footprint" "antmicro-footprints:R_0402_1005Metric"
+		(property "Footprint" "antmicro-footprints:R_0603_1608Metric"
 			(at 203.2 45.72 0)
 			(effects
@@
 			)
 		)
-		(property "Description" "SMD Chip Resistor, 120 ohm, ± 1%, 63 mW, 0402 [1005 Metric], Thick Film, General Purpose"
+		(property "Description" "SMD Chip Resistor, 120 ohm, ± 1%, 100 mW, 0603 [1608 Metric], Thick Film, General Purpose"
 			(at 218.44 66.04 0)
 			(effects
@@
 			)
 		)
-		(property "MPN" "CR0402-FX-1200GLF"
+		(property "MPN" "CR0603-FX-1200ELF"
 			(at 198.12 45.72 0)
 			(effects
@@
 	)
 	(symbol
-		(lib_id "antmicroResistors0402:R_120R_0402")
+		(lib_id "antmicroResistors0603:R_120R_0603")
 		(at 104.14 157.48 270)
 		(mirror x)
@@
 			)
 		)
-		(property "Value" "R_120R_0402"
+		(property "Value" "R_120R_0603"
 			(at 91.44 137.16 0)
 			(effects
@@
 			)
 		)
-		(property "Footprint" "antmicro-footprints:R_0402_1005Metric"
+		(property "Footprint" "antmicro-footprints:R_0603_1608Metric"
 			(at 88.9 137.16 0)
 			(effects
@@
 			)
 		)
-		(property "Description" "SMD Chip Resistor, 120 ohm, ± 1%, 63 mW, 0402 [1005 Metric], Thick Film, General Purpose"
+		(property "Description" "SMD Chip Resistor, 120 ohm, ± 1%, 100 mW, 0603 [1608 Metric], Thick Film, General Purpose"
 			(at 104.14 157.48 0)
 			(effects
@@
 			)
 		)
-		(property "MPN" "CR0402-FX-1200GLF"
+		(property "MPN" "CR0603-FX-1200ELF"
 			(at 83.82 137.16 0)
 			(effects
@@
 	)
 	(symbol
-		(lib_id "antmicroResistors0402:R_120R_0402")
+		(lib_id "antmicroResistors0603:R_120R_0603")
 		(at 218.44 88.9 270)
 		(mirror x)
@@
 			)
 		)
-		(property "Value" "R_120R_0402"
+		(property "Value" "R_120R_0603"
 			(at 205.74 68.58 0)
 			(effects
@@
 			)
 		)
-		(property "Footprint" "antmicro-footprints:R_0402_1005Metric"
+		(property "Footprint" "antmicro-footprints:R_0603_1608Metric"
 			(at 203.2 68.58 0)
 			(effects
@@
 			)
 		)
-		(property "Description" "SMD Chip Resistor, 120 ohm, ± 1%, 63 mW, 0402 [1005 Metric], Thick Film, General Purpose"
+		(property "Description" "SMD Chip Resistor, 120 ohm, ± 1%, 100 mW, 0603 [1608 Metric], Thick Film, General Purpose"
 			(at 218.44 88.9 0)
 			(effects
@@
 			)
 		)
-		(property "MPN" "CR0402-FX-1200GLF"
+		(property "MPN" "CR0603-FX-1200ELF"
 			(at 198.12 68.58 0)
 			(effects
@@
 	)
 	(symbol
-		(lib_id "antmicroResistors0402:R_120R_0402")
+		(lib_id "antmicroResistors0603:R_120R_0603")
 		(at 218.44 134.62 270)
 		(mirror x)
@@
 			)
 		)
-		(property "Value" "R_120R_0402"
+		(property "Value" "R_120R_0603"
 			(at 205.74 114.3 0)
 			(effects
@@
 			)
 		)
-		(property "Footprint" "antmicro-footprints:R_0402_1005Metric"
+		(property "Footprint" "antmicro-footprints:R_0603_1608Metric"
 			(at 203.2 114.3 0)
 			(effects
@@
 			)
 		)
-		(property "Description" "SMD Chip Resistor, 120 ohm, ± 1%, 63 mW, 0402 [1005 Metric], Thick Film, General Purpose"
+		(property "Description" "SMD Chip Resistor, 120 ohm, ± 1%, 100 mW, 0603 [1608 Metric], Thick Film, General Purpose"
 			(at 218.44 134.62 0)
 			(effects
@@
 			)
 		)
-		(property "MPN" "CR0402-FX-1200GLF"
+		(property "MPN" "CR0603-FX-1200ELF"
 			(at 198.12 114.3 0)
 			(effects
@@
 	)
 	(symbol
-		(lib_id "antmicroResistors0402:R_120R_0402")
+		(lib_id "antmicroResistors0603:R_120R_0603")
 		(at 218.44 157.48 270)
 		(mirror x)
@@
 			)
 		)
-		(property "Value" "R_120R_0402"
+		(property "Value" "R_120R_0603"
 			(at 205.74 137.16 0)
 			(effects
@@
 			)
 		)
-		(property "Footprint" "antmicro-footprints:R_0402_1005Metric"
+		(property "Footprint" "antmicro-footprints:R_0603_1608Metric"
 			(at 203.2 137.16 0)
 			(effects
@@
 			)
 		)
-		(property "Description" "SMD Chip Resistor, 120 ohm, ± 1%, 63 mW, 0402 [1005 Metric], Thick Film, General Purpose"
+		(property "Description" "SMD Chip Resistor, 120 ohm, ± 1%, 100 mW, 0603 [1608 Metric], Thick Film, General Purpose"
 			(at 218.44 157.48 0)
 			(effects
@@
 			)
 		)
-		(property "MPN" "CR0402-FX-1200GLF"
+		(property "MPN" "CR0603-FX-1200ELF"
 			(at 198.12 137.16 0)
 			(effects
@@
 	)
 	(symbol
-		(lib_id "antmicroResistors0402:R_120R_0402")
+		(lib_id "antmicroResistors0603:R_120R_0603")
 		(at 104.14 111.76 270)
 		(mirror x)
@@
 			)
 		)
-		(property "Value" "R_120R_0402"
+		(property "Value" "R_120R_0603"
 			(at 91.44 91.44 0)
 			(effects
@@
 			)
 		)
-		(property "Footprint" "antmicro-footprints:R_0402_1005Metric"
+		(property "Footprint" "antmicro-footprints:R_0603_1608Metric"
 			(at 88.9 91.44 0)
 			(effects
@@
 			)
 		)
-		(property "Description" "SMD Chip Resistor, 120 ohm, ± 1%, 63 mW, 0402 [1005 Metric], Thick Film, General Purpose"
+		(property "Description" "SMD Chip Resistor, 120 ohm, ± 1%, 100 mW, 0603 [1608 Metric], Thick Film, General Purpose"
 			(at 104.14 111.76 0)
 			(effects
@@
 			)
 		)
-		(property "MPN" "CR0402-FX-1200GLF"
+		(property "MPN" "CR0603-FX-1200ELF"
 			(at 83.82 91.44 0)
 			(effects
@@
 	)
 	(symbol
-		(lib_id "antmicroResistors0402:R_120R_0402")
+		(lib_id "antmicroResistors0603:R_120R_0603")
 		(at 104.14 134.62 270)
 		(mirror x)
@@
 			)
 		)
-		(property "Value" "R_120R_0402"
+		(property "Value" "R_120R_0603"
 			(at 91.44 114.3 0)
 			(effects
@@
 			)
 		)
-		(property "Footprint" "antmicro-footprints:R_0402_1005Metric"
+		(property "Footprint" "antmicro-footprints:R_0603_1608Metric"
 			(at 88.9 114.3 0)
 			(effects
@@
 			)
 		)
-		(property "Description" "SMD Chip Resistor, 120 ohm, ± 1%, 63 mW, 0402 [1005 Metric], Thick Film, General Purpose"
+		(property "Description" "SMD Chip Resistor, 120 ohm, ± 1%, 100 mW, 0603 [1608 Metric], Thick Film, General Purpose"
 			(at 104.14 134.62 0)
 			(effects
@@
 			)
 		)
-		(property "MPN" "CR0402-FX-1200GLF"
+		(property "MPN" "CR0603-FX-1200ELF"
 			(at 83.82 114.3 0)
 			(effects
@@
 	)
 	(symbol
-		(lib_id "antmicroResistors0402:R_120R_0402")
+		(lib_id "antmicroResistors0603:R_120R_0603")
 		(at 104.14 88.9 270)
 		(mirror x)
@@
 			)
 		)
-		(property "Value" "R_120R_0402"
+		(property "Value" "R_120R_0603"
 			(at 91.44 68.58 0)
 			(effects
@@
 			)
 		)
-		(property "Footprint" "antmicro-footprints:R_0402_1005Metric"
+		(property "Footprint" "antmicro-footprints:R_0603_1608Metric"
 			(at 88.9 68.58 0)
 			(effects
@@
 			)
 		)
-		(property "Description" "SMD Chip Resistor, 120 ohm, ± 1%, 63 mW, 0402 [1005 Metric], Thick Film, General Purpose"
+		(property "Description" "SMD Chip Resistor, 120 ohm, ± 1%, 100 mW, 0603 [1608 Metric], Thick Film, General Purpose"
 			(at 104.14 88.9 0)
 			(effects
@@
 			)
 		)
-		(property "MPN" "CR0402-FX-1200GLF"
+		(property "MPN" "CR0603-FX-1200ELF"
 			(at 83.82 68.58 0)
 			(effects
